File: PCBdesign/teamNACHOrev1.sch (EAGLE design)
At the start: 15 parts, among them Q2 TK40E06N1

Commit message: Slowly but surely
Slowly adding more components to schematic. still not sure how to do
atmega correctly
Parts:
- added R3: 12, rcl:R-US_M0805
- added X1: (no value), con-berg:PN87520
Connections:
- new net N$10: C6.2, U$2.SEC2
- new net N$8: R3.1
- new net N$9: R3.2
- net +5V: now also X1.1
- net GND: now also Q2.S, X1.4
Changed lines of the file:
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@@
 <part name="D2" library="diode" deviceset="1N4004" device=""/>
 <part name="C6" library="rcl" deviceset="C-US" device="C0805" value="10u"/>
+<part name="R3" library="rcl" deviceset="R-US_" device="M0805" value="12"/>
+<part name="X1" library="con-berg" deviceset="PN87520" device=""/>
+<part name="P+6" library="supply1" deviceset="+5V" device=""/>
+<part name="SUPPLY8" library="supply2" deviceset="GND" device=""/>
+<part name="SUPPLY9" library="supply2" deviceset="GND" device=""/>
 </parts>
 <sheets>
@@
 <instance part="D2" gate="1" x="110.49" y="-16.51"/>
 <instance part="C6" gate="G$1" x="127" y="-19.05"/>
+<instance part="R3" gate="G$1" x="163.83" y="-16.51"/>
+<instance part="X1" gate="G$1" x="-12.7" y="76.2" rot="R180"/>
+<instance part="P+6" gate="1" x="-2.54" y="76.2"/>
+<instance part="SUPPLY8" gate="GND" x="3.81" y="76.2"/>
+<instance part="SUPPLY9" gate="GND" x="63.5" y="-50.8"/>
 </instances>
 <busses>
@@
 <wire x1="123.19" y1="0" x2="134.62" y2="0" width="0.1524" layer="91"/>
 <pinref part="SUPPLY7" gate="GND" pin="GND"/>
+</segment>
+<segment>
+<pinref part="X1" gate="G$1" pin="4"/>
+<wire x1="-10.16" y1="78.74" x2="3.81" y2="78.74" width="0.1524" layer="91"/>
+<pinref part="SUPPLY8" gate="GND" pin="GND"/>
+</segment>
+<segment>
+<pinref part="Q2" gate="G$1" pin="S"/>
+<wire x1="63.5" y1="-45.72" x2="63.5" y2="-48.26" width="0.1524" layer="91"/>
+<pinref part="SUPPLY9" gate="GND" pin="GND"/>
 </segment>
 </net>
@@
 <junction x="45.72" y="-16.51"/>
 </segment>
+<segment>
+<pinref part="X1" gate="G$1" pin="1"/>
+<wire x1="-10.16" y1="71.12" x2="-2.54" y2="71.12" width="0.1524" layer="91"/>
+<pinref part="P+6" gate="1" pin="+5V"/>
+<wire x1="-2.54" y1="71.12" x2="-2.54" y2="73.66" width="0.1524" layer="91"/>
+</segment>
 </net>
 <net name="SCK" class="0">
@@
 <pinref part="C6" gate="G$1" pin="1"/>
 <wire x1="113.03" y1="-16.51" x2="127" y2="-16.51" width="0.1524" layer="91"/>
-</segment>
-</net>
+<wire x1="127" y1="-16.51" x2="134.62" y2="-16.51" width="0.1524" layer="91"/>
+</segment>
+</net>
+<net name="N$8" class="0">
+<segment>
+<pinref part="R3" gate="G$1" pin="1"/>
+<wire x1="154.94" y1="-16.51" x2="158.75" y2="-16.51" width="0.1524" layer="91"/>
+</segment>
+</net>
+<net name="N$9" class="0">
+<segment>
+<pinref part="R3" gate="G$1" pin="2"/>
+<wire x1="168.91" y1="-16.51" x2="172.72" y2="-16.51" width="0.1524" layer="91"/>
+<wire x1="172.72" y1="-16.51" x2="172.72" y2="-24.13" width="0.1524" layer="91"/>
+<wire x1="172.72" y1="-24.13" x2="144.78" y2="-24.13" width="0.1524" layer="91"/>
+</segment>
+</net>
+<net name="N$10" class="0">
+<segment>
+<pinref part="U$2" gate="G$1" pin="SEC2"/>
+<wire x1="96.52" y1="-22.86" x2="100.33" y2="-22.86" width="0.1524" layer="91"/>
+<wire x1="100.33" y1="-22.86" x2="100.33" y2="-26.67" width="0.1524" layer="91"/>
+<wire x1="100.33" y1="-26.67" x2="127" y2="-26.67" width="0.1524" layer="91"/>
+<pinref part="C6" gate="G$1" pin="2"/>
+<wire x1="127" y1="-26.67" x2="177.8" y2="-26.67" width="0.1524" layer="91"/>
+<wire x1="127" y1="-24.13" x2="127" y2="-26.67" width="0.1524" layer="91"/>
+<junction x="127" y="-26.67"/>
+</segment>
+</net>

Commit message: Fixed USB
Flipped which pins on USB are ground and power. Also may have to make
own lib for LM317, they don’t have the correct pcb package we need.
Connections:
- net +5V: now also X1.4; no longer X1.1
- net GND: now also X1.1; no longer X1.4
Other:
- moved on the sheet: X1
Changed lines of the file:
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@@
 <part name="C6" library="rcl" deviceset="C-US" device="C0805" value="10u"/>
 <part name="R3" library="rcl" deviceset="R-US_" device="M0805" value="12"/>
+<part name="SUPPLY9" library="supply2" deviceset="GND" device=""/>
 <part name="X1" library="con-berg" deviceset="PN87520" device=""/>
 <part name="P+6" library="supply1" deviceset="+5V" device=""/>
 <part name="SUPPLY8" library="supply2" deviceset="GND" device=""/>
-<part name="SUPPLY9" library="supply2" deviceset="GND" device=""/>
 </parts>
 <sheets>
@@
 <instance part="C6" gate="G$1" x="127" y="-19.05"/>
 <instance part="R3" gate="G$1" x="163.83" y="-16.51"/>
-<instance part="X1" gate="G$1" x="-12.7" y="76.2" rot="R180"/>
-<instance part="P+6" gate="1" x="-2.54" y="76.2"/>
-<instance part="SUPPLY8" gate="GND" x="3.81" y="76.2"/>
 <instance part="SUPPLY9" gate="GND" x="63.5" y="-50.8"/>
+<instance part="X1" gate="G$1" x="-5.08" y="68.58" rot="R180"/>
+<instance part="P+6" gate="1" x="5.08" y="76.2"/>
+<instance part="SUPPLY8" gate="GND" x="5.08" y="60.96"/>
 </instances>
 <busses>
@@
 </segment>
 <segment>
-<pinref part="X1" gate="G$1" pin="4"/>
-<wire x1="-10.16" y1="78.74" x2="3.81" y2="78.74" width="0.1524" layer="91"/>
-<pinref part="SUPPLY8" gate="GND" pin="GND"/>
-</segment>
-<segment>
 <pinref part="Q2" gate="G$1" pin="S"/>
 <wire x1="63.5" y1="-45.72" x2="63.5" y2="-48.26" width="0.1524" layer="91"/>
 <pinref part="SUPPLY9" gate="GND" pin="GND"/>
+</segment>
+<segment>
+<pinref part="X1" gate="G$1" pin="1"/>
+<wire x1="-2.54" y1="63.5" x2="5.08" y2="63.5" width="0.1524" layer="91"/>
+<pinref part="SUPPLY8" gate="GND" pin="GND"/>
 </segment>
 </net>
@@
 </segment>
 <segment>
-<pinref part="X1" gate="G$1" pin="1"/>
-<wire x1="-10.16" y1="71.12" x2="-2.54" y2="71.12" width="0.1524" layer="91"/>
+<pinref part="X1" gate="G$1" pin="4"/>
+<wire x1="-2.54" y1="71.12" x2="5.08" y2="71.12" width="0.1524" layer="91"/>
+<wire x1="5.08" y1="71.12" x2="5.08" y2="73.66" width="0.1524" layer="91"/>
 <pinref part="P+6" gate="1" pin="+5V"/>
-<wire x1="-2.54" y1="71.12" x2="-2.54" y2="73.66" width="0.1524" layer="91"/>
 </segment>
 </net>
