File: PCBdesign/teamNACHOrev1.sch (EAGLE design)
At the start: 47 parts, among them IC1 7805TV, Q2 TK40E06N1, Q3 TK40E06N1, U2 ATTINY85V-10SU, X2 1751248, X3 1751251

Commit message: hur ya go
asdfasdf
Parts:
- added C11: 10u, rcl:C-USC0805
- added C12: 0.1u, rcl:C-USC0805
- added LED2: (no value), eagle-ltspice:LED_ELD260
- added R12: 470, rcl:R-US_M0805
- R8: value 100 -> 30k
- R9: value 100 -> 10k
Connections:
- removed net N$11: X2-2.K
- new net SCK-AT: JP2.3, U2.PB3
- net +5V: now also C11.1, C12.1
- net 5: now also R12.1
- net FB: now also R3.2, U$3.ADJ, X2-1.K
- net GND: now also C11.2, C12.2, LED2.C; no longer OK1.C
- net GND_S: now also OK1.C, X2-2.K
- net N$8: now also U$3.VOUT
- net N$9: now also LED2.A, R12.2; no longer R3.2, X2-1.K
- net VFB: now also U2.PB4; no longer JP2.3, U2.PB3
Other:
- moved on the sheet: X2-2
Changed lines of the file:
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@@
 <part name="P+5" library="supply1" deviceset="+5V" device=""/>
 <part name="SUPPLY15" library="supply2" deviceset="GND" device=""/>
-<part name="GND3" library="supply1" deviceset="GND" device=""/>
 <part name="R7" library="rcl" deviceset="R-US_" device="M0805" value="1k"/>
 <part name="JP2" library="avr-7" deviceset="AVR-ISP-6" device="VERT"/>
@@
 <part name="C9" library="rcl" deviceset="C-US" device="C0805" value="0.33u"/>
 <part name="C10" library="rcl" deviceset="C-US" device="C0805" value="0.1u"/>
-<part name="R8" library="resistor" deviceset="R-US_" device="R0805" value="100"/>
-<part name="R9" library="resistor" deviceset="R-US_" device="R0805" value="100"/>
+<part name="R8" library="resistor" deviceset="R-US_" device="R0805" value="30k"/>
+<part name="R9" library="resistor" deviceset="R-US_" device="R0805" value="10k"/>
 <part name="S1" library="switch" deviceset="55?" device="01"/>
 <part name="S2" library="switch" deviceset="55?" device="01"/>
@@
 <part name="SUPPLY11" library="supply2" deviceset="GND" device=""/>
 <part name="SUPPLY12" library="supply2" deviceset="GND" device=""/>
+<part name="C11" library="rcl" deviceset="C-US" device="C0805" value="10u"/>
+<part name="C12" library="rcl" deviceset="C-US" device="C0805" value="0.1u"/>
+<part name="LED2" library="eagle-ltspice" deviceset="LED_E" device="LD260"/>
+<part name="R12" library="rcl" deviceset="R-US_" device="M0805" value="470"/>
+<part name="SUPPLY14" library="supply2" deviceset="GND" device=""/>
 </parts>
 <sheets>
@@
 <instance part="SUPPLY9" gate="GND" x="63.5" y="-50.8"/>
 <instance part="X1" gate="G$1" x="-5.08" y="68.58" rot="R180"/>
-<instance part="P+6" gate="1" x="22.86" y="78.74"/>
+<instance part="P+6" gate="1" x="39.37" y="78.74"/>
 <instance part="SUPPLY8" gate="GND" x="5.08" y="60.96"/>
 <instance part="U$3" gate="G$1" x="147.32" y="-16.51"/>
 <instance part="X2" gate="-1" x="194.31" y="-16.51"/>
-<instance part="X2" gate="-2" x="194.31" y="-24.13"/>
+<instance part="X2" gate="-2" x="194.31" y="-22.86"/>
 <instance part="X3" gate="-1" x="194.31" y="6.35"/>
 <instance part="X3" gate="-2" x="194.31" y="-1.27"/>
@@
 <instance part="F1" gate="G$1" x="6.35" y="71.12"/>
 <instance part="D3" gate="1" x="15.24" y="66.04" rot="R90"/>
-<instance part="U$4" gate="G$1" x="33.02" y="71.12"/>
+<instance part="U$4" gate="G$1" x="49.53" y="71.12"/>
 <instance part="U$5" gate="G$1" x="95.25" y="-71.12"/>
 <instance part="Q3" gate="G$1" x="60.96" y="-76.2"/>
@@
 <instance part="P+5" gate="1" x="151.13" y="20.32"/>
 <instance part="SUPPLY15" gate="GND" x="161.29" y="43.18" rot="R180"/>
-<instance part="GND3" gate="1" x="181.61" y="40.64" rot="R90"/>
 <instance part="R7" gate="G$1" x="179.07" y="27.94" rot="R90"/>
 <instance part="JP2" gate="G$1" x="256.54" y="-55.88"/>
@@
 <instance part="SUPPLY11" gate="GND" x="184.15" y="69.85"/>
 <instance part="SUPPLY12" gate="GND" x="184.15" y="55.88"/>
+<instance part="C11" gate="G$1" x="22.86" y="68.58"/>
+<instance part="C12" gate="G$1" x="30.48" y="68.58"/>
+<instance part="LED2" gate="G$1" x="66.04" y="83.82" rot="R180"/>
+<instance part="R12" gate="G$1" x="66.04" y="76.2" rot="R90"/>
+<instance part="SUPPLY14" gate="GND" x="66.04" y="91.44" rot="R180"/>
 </instances>
 <busses>
@@
 <pinref part="D3" gate="1" pin="A"/>
 <wire x1="5.08" y1="63.5" x2="15.24" y2="63.5" width="0.1524" layer="91"/>
+<pinref part="C11" gate="G$1" pin="2"/>
+<wire x1="15.24" y1="63.5" x2="22.86" y2="63.5" width="0.1524" layer="91"/>
+<pinref part="C12" gate="G$1" pin="2"/>
+<wire x1="30.48" y1="63.5" x2="22.86" y2="63.5" width="0.1524" layer="91"/>
 </segment>
 <segment>
@@
 </segment>
 <segment>
-<pinref part="OK1" gate="G$1" pin="C"/>
-<pinref part="GND3" gate="1" pin="GND"/>
-</segment>
-<segment>
 <pinref part="SV1" gate="1" pin="2"/>
 <pinref part="SUPPLY16" gate="GND" pin="GND"/>
@@
 <wire x1="179.07" y1="58.42" x2="184.15" y2="58.42" width="0.1524" layer="91"/>
 <pinref part="SUPPLY12" gate="GND" pin="GND"/>
+</segment>
+<segment>
+<pinref part="LED2" gate="G$1" pin="C"/>
+<pinref part="SUPPLY14" gate="GND" pin="GND"/>
 </segment>
 </net>
@@
 </segment>
 <segment>
-<wire x1="22.86" y1="71.12" x2="22.86" y2="76.2" width="0.1524" layer="91"/>
+<wire x1="39.37" y1="71.12" x2="39.37" y2="76.2" width="0.1524" layer="91"/>
 <pinref part="P+6" gate="1" pin="+5V"/>
 <pinref part="F1" gate="G$1" pin="2"/>
@@
 <pinref part="D3" gate="1" pin="C"/>
 <wire x1="15.24" y1="71.12" x2="22.86" y2="71.12" width="0.1524" layer="91"/>
+<wire x1="22.86" y1="71.12" x2="30.48" y2="71.12" width="0.1524" layer="91"/>
+<wire x1="30.48" y1="71.12" x2="39.37" y2="71.12" width="0.1524" layer="91"/>
 <wire x1="15.24" y1="68.58" x2="15.24" y2="71.12" width="0.1524" layer="91"/>
 <junction x="15.24" y="71.12"/>
 <pinref part="U$4" gate="G$1" pin="1"/>
+<junction x="39.37" y="71.12"/>
+<pinref part="C11" gate="G$1" pin="1"/>
 <junction x="22.86" y="71.12"/>
+<pinref part="C12" gate="G$1" pin="1"/>
+<junction x="30.48" y="71.12"/>
 </segment>
 <segment>
@@
 <pinref part="D2" gate="1" pin="A"/>
 <wire x1="100.33" y1="-16.51" x2="107.95" y2="-16.51" width="0.1524" layer="91"/>
+<junction x="100.33" y="-20.32"/>
 </segment>
 </net>
@@
 <pinref part="R3" gate="G$1" pin="1"/>
 <wire x1="163.83" y1="-16.51" x2="167.64" y2="-16.51" width="0.1524" layer="91"/>
-</segment>
-</net>
-<net name="N$9" class="0">
-<segment>
-<pinref part="R3" gate="G$1" pin="2"/>
-<wire x1="177.8" y1="-16.51" x2="181.61" y2="-16.51" width="0.1524" layer="91"/>
-<wire x1="181.61" y1="-16.51" x2="181.61" y2="-24.13" width="0.1524" layer="91"/>
-<wire x1="181.61" y1="-24.13" x2="148.59" y2="-24.13" width="0.1524" layer="91"/>
-<pinref part="X2" gate="-1" pin="K"/>
-<wire x1="181.61" y1="-16.51" x2="191.77" y2="-16.51" width="0.1524" layer="91"/>
-<junction x="181.61" y="-16.51"/>
-</segment>
-</net>
-<net name="N$11" class="0">
-<segment>
-<pinref part="X2" gate="-2" pin="K"/>
-<wire x1="191.77" y1="-24.13" x2="191.77" y2="-26.67" width="0.1524" layer="91"/>
+<pinref part="U$3" gate="G$1" pin="VOUT"/>
 </segment>
 </net>
@@
 <label x="130.81" y="-35.56" size="1.778" layer="95"/>
 </segment>
+<segment>
+<pinref part="R3" gate="G$1" pin="2"/>
+<wire x1="177.8" y1="-16.51" x2="181.61" y2="-16.51" width="0.1524" layer="91"/>
+<wire x1="181.61" y1="-16.51" x2="181.61" y2="-24.13" width="0.1524" layer="91"/>
+<wire x1="181.61" y1="-24.13" x2="148.59" y2="-24.13" width="0.1524" layer="91"/>
+<pinref part="U$3" gate="G$1" pin="ADJ"/>
+<pinref part="X2" gate="-1" pin="K"/>
+<wire x1="181.61" y1="-16.51" x2="191.77" y2="-16.51" width="0.1524" layer="91"/>
+<junction x="181.61" y="-16.51"/>
+<label x="182.88" y="-16.51" size="1.778" layer="95"/>
+</segment>
 </net>
 <net name="AT-PWM" class="0">
@@
 <segment>
 <pinref part="U$4" gate="G$1" pin="1A"/>
-<wire x1="45.72" y1="71.12" x2="55.88" y2="71.12" width="0.1524" layer="91"/>
-<label x="50.8" y="71.12" size="1.778" layer="95"/>
+<wire x1="62.23" y1="71.12" x2="66.04" y2="71.12" width="0.1524" layer="91"/>
+<label x="71.12" y="71.12" size="1.778" layer="95"/>
+<pinref part="R12" gate="G$1" pin="1"/>
+<junction x="66.04" y="71.12"/>
+<wire x1="66.04" y1="71.12" x2="72.39" y2="71.12" width="0.1524" layer="91"/>
 </segment>
 <segment>
@@
 <junction x="127" y="-26.67"/>
 <label x="135.89" y="-26.67" size="1.778" layer="95"/>
+<pinref part="X2" gate="-2" pin="K"/>
+<wire x1="191.77" y1="-22.86" x2="191.77" y2="-26.67" width="0.1524" layer="91"/>
+<junction x="191.77" y="-26.67"/>
+<junction x="100.33" y="-22.86"/>
 </segment>
 <segment>
@@
 <label x="163.83" y="-35.56" size="1.778" layer="95"/>
 </segment>
+<segment>
+<pinref part="OK1" gate="G$1" pin="C"/>
+<wire x1="179.07" y1="40.64" x2="186.69" y2="40.64" width="0.1524" layer="91"/>
+<label x="180.34" y="40.64" size="1.778" layer="95"/>
+</segment>
 </net>
 <net name="VFB" class="0">
@@
 </segment>
 <segment>
-<pinref part="U2" gate="A" pin="PB3"/>
-<wire x1="229.87" y1="-59.69" x2="241.3" y2="-59.69" width="0.1524" layer="91"/>
-<label x="236.22" y="-59.69" size="1.778" layer="95"/>
-<label x="187.96" y="-16.51" size="1.778" layer="95"/>
-<wire x1="241.3" y1="-59.69" x2="241.3" y2="-55.88" width="0.1524" layer="91"/>
-<pinref part="JP2" gate="G$1" pin="3"/>
-<wire x1="241.3" y1="-55.88" x2="251.46" y2="-55.88" width="0.1524" layer="91"/>
+<pinref part="U2" gate="A" pin="PB4"/>
+<wire x1="229.87" y1="-62.23" x2="241.3" y2="-62.23" width="0.1524" layer="91"/>
+<label x="234.95" y="-62.23" size="1.778" layer="95"/>
 </segment>
 </net>
@@
 </segment>
 </net>
+<net name="SCK-AT" class="0">
+<segment>
+<pinref part="U2" gate="A" pin="PB3"/>
+<wire x1="229.87" y1="-59.69" x2="241.3" y2="-59.69" width="0.1524" layer="91"/>
+<wire x1="241.3" y1="-59.69" x2="241.3" y2="-55.88" width="0.1524" layer="91"/>
+<pinref part="JP2" gate="G$1" pin="3"/>
+<wire x1="241.3" y1="-55.88" x2="251.46" y2="-55.88" width="0.1524" layer="91"/>
+<label x="234.95" y="-59.69" size="1.778" layer="95"/>
+</segment>
+</net>
+<net name="N$9" class="0">
+<segment>
+<pinref part="LED2" gate="G$1" pin="A"/>
+<pinref part="R12" gate="G$1" pin="2"/>
+</segment>
+</net>

Commit message: HERE YOU GO ADAM
Parts:
- removed R10, R11: 1k, rcl:R-US_R0805
- removed S1, S2: 5501, switch:5501
- added TP1, TP2, TP3, TP4, TP5, TP6: PTR1PAD1-20, testpad:PTR1PAD1-20
- SV1: device con-lstb:MA04-1 -> con-lsta:FE06-1
Connections:
- new net N$11: TP3.TP, X3-2.K
- net +5V: no longer S1.1A, S2.1A
- net FB-CGRD: now also TP2.TP
- net GND: now also TP6.TP; no longer R10.1, R11.1
- net GND_S: now also TP5.TP
- net LED-CLK: now also SV1.3
- net LED-DAT: now also SV1.4
- net PB_1: now also SV1.5; no longer R10.2, S1.NO
- net PB_2: now also SV1.6; no longer R11.2, S2.NO
- net POT: now also TP1.TP; no longer X3-2.K
- net VFB: now also TP4.TP
Other:
- note added: "FEMALE PINS TO LCD PCB"
Changed lines of the file:
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@@
 <part name="R7" library="rcl" deviceset="R-US_" device="M0805" value="1k"/>
 <part name="JP2" library="avr-7" deviceset="AVR-ISP-6" device="VERT"/>
-<part name="SV1" library="con-lstb" deviceset="MA04-1" device=""/>
 <part name="P+8" library="supply1" deviceset="+5V" device=""/>
 <part name="SUPPLY16" library="supply2" deviceset="GND" device=""/>
@@
 <part name="R8" library="resistor" deviceset="R-US_" device="R0805" value="30k"/>
 <part name="R9" library="resistor" deviceset="R-US_" device="R0805" value="10k"/>
-<part name="S1" library="switch" deviceset="55?" device="01"/>
-<part name="S2" library="switch" deviceset="55?" device="01"/>
-<part name="P+9" library="supply1" deviceset="+5V" device=""/>
-<part name="P+10" library="supply1" deviceset="+5V" device=""/>
-<part name="R10" library="rcl" deviceset="R-US_" device="R0805" value="1k"/>
-<part name="R11" library="rcl" deviceset="R-US_" device="R0805" value="1k"/>
-<part name="SUPPLY11" library="supply2" deviceset="GND" device=""/>
-<part name="SUPPLY12" library="supply2" deviceset="GND" device=""/>
 <part name="C11" library="rcl" deviceset="C-US" device="C0805" value="10u"/>
 <part name="C12" library="rcl" deviceset="C-US" device="C0805" value="0.1u"/>
@@
 <part name="R12" library="rcl" deviceset="R-US_" device="M0805" value="470"/>
 <part name="SUPPLY14" library="supply2" deviceset="GND" device=""/>
+<part name="TP1" library="testpad" deviceset="PTR1" device="PAD1-20"/>
+<part name="TP2" library="testpad" deviceset="PTR1" device="PAD1-20"/>
+<part name="TP3" library="testpad" deviceset="PTR1" device="PAD1-20"/>
+<part name="TP4" library="testpad" deviceset="PTR1" device="PAD1-20"/>
+<part name="TP5" library="testpad" deviceset="PTR1" device="PAD1-20"/>
+<part name="TP6" library="testpad" deviceset="PTR1" device="PAD1-20"/>
+<part name="SV1" library="con-lsta" deviceset="FE06-1" device=""/>
 </parts>
 <sheets>
 <sheet>
 <plain>
+<text x="119.38" y="78.74" size="1.778" layer="91">FEMALE PINS
+TO LCD PCB</text>
 </plain>
 <instances>
@@
 <instance part="R7" gate="G$1" x="179.07" y="27.94" rot="R90"/>
 <instance part="JP2" gate="G$1" x="256.54" y="-55.88"/>
-<instance part="SV1" gate="1" x="120.65" y="69.85" rot="R180"/>
 <instance part="P+8" gate="1" x="113.03" y="81.28"/>
 <instance part="SUPPLY16" gate="GND" x="105.41" y="74.93" rot="R180"/>
@@
 <instance part="R8" gate="G$1" x="140.97" y="-35.56" rot="R180"/>
 <instance part="R9" gate="G$1" x="157.48" y="-35.56" rot="R180"/>
-<instance part="S1" gate="G$1" x="156.21" y="74.93"/>
-<instance part="S2" gate="G$1" x="156.21" y="60.96"/>
-<instance part="P+9" gate="1" x="144.78" y="77.47"/>
-<instance part="P+10" gate="1" x="144.78" y="63.5"/>
-<instance part="R10" gate="G$1" x="173.99" y="72.39" rot="R180"/>
-<instance part="R11" gate="G$1" x="173.99" y="58.42" rot="R180"/>
-<instance part="SUPPLY11" gate="GND" x="184.15" y="69.85"/>
-<instance part="SUPPLY12" gate="GND" x="184.15" y="55.88"/>
 <instance part="C11" gate="G$1" x="22.86" y="68.58"/>
 <instance part="C12" gate="G$1" x="30.48" y="68.58"/>
@@
 <instance part="R12" gate="G$1" x="66.04" y="76.2" rot="R90"/>
 <instance part="SUPPLY14" gate="GND" x="66.04" y="91.44" rot="R180"/>
+<instance part="TP1" gate="G$1" x="120.65" y="46.99" rot="R90"/>
+<instance part="TP2" gate="G$1" x="120.65" y="49.53" rot="R90"/>
+<instance part="TP3" gate="G$1" x="189.23" y="-1.27" rot="R270"/>
+<instance part="TP4" gate="G$1" x="149.86" y="-38.1"/>
+<instance part="TP5" gate="G$1" x="118.11" y="-29.21"/>
+<instance part="TP6" gate="G$1" x="11.43" y="60.96"/>
+<instance part="SV1" gate="G$1" x="120.65" y="69.85" rot="R180"/>
 </instances>
 <busses>
@@
 <pinref part="SUPPLY8" gate="GND" pin="GND"/>
 <pinref part="D3" gate="1" pin="A"/>
-<wire x1="5.08" y1="63.5" x2="15.24" y2="63.5" width="0.1524" layer="91"/>
+<wire x1="5.08" y1="63.5" x2="11.43" y2="63.5" width="0.1524" layer="91"/>
 <pinref part="C11" gate="G$1" pin="2"/>
+<wire x1="11.43" y1="63.5" x2="15.24" y2="63.5" width="0.1524" layer="91"/>
 <wire x1="15.24" y1="63.5" x2="22.86" y2="63.5" width="0.1524" layer="91"/>
 <pinref part="C12" gate="G$1" pin="2"/>
 <wire x1="30.48" y1="63.5" x2="22.86" y2="63.5" width="0.1524" layer="91"/>
+<pinref part="TP6" gate="G$1" pin="TP"/>
+<junction x="11.43" y="63.5"/>
 </segment>
 <segment>
@@
 </segment>
 <segment>
-<pinref part="SV1" gate="1" pin="2"/>
 <pinref part="SUPPLY16" gate="GND" pin="GND"/>
 <wire x1="105.41" y1="72.39" x2="113.03" y2="72.39" width="0.1524" layer="91"/>
-</segment>
-<segment>
-<pinref part="R10" gate="G$1" pin="1"/>
-<wire x1="179.07" y1="72.39" x2="184.15" y2="72.39" width="0.1524" layer="91"/>
-<pinref part="SUPPLY11" gate="GND" pin="GND"/>
-</segment>
-<segment>
-<pinref part="R11" gate="G$1" pin="1"/>
-<wire x1="179.07" y1="58.42" x2="184.15" y2="58.42" width="0.1524" layer="91"/>
-<pinref part="SUPPLY12" gate="GND" pin="GND"/>
+<pinref part="SV1" gate="G$1" pin="2"/>
 </segment>
 <segment>
@@
 </segment>
 <segment>
-<pinref part="SV1" gate="1" pin="1"/>
 <pinref part="P+8" gate="1" pin="+5V"/>
 <wire x1="113.03" y1="78.74" x2="113.03" y2="74.93" width="0.1524" layer="91"/>
-</segment>
-<segment>
-<pinref part="S1" gate="G$1" pin="1A"/>
-<wire x1="151.13" y1="74.93" x2="144.78" y2="74.93" width="0.1524" layer="91"/>
-<pinref part="P+9" gate="1" pin="+5V"/>
-</segment>
-<segment>
-<pinref part="S2" gate="G$1" pin="1A"/>
-<wire x1="151.13" y1="60.96" x2="144.78" y2="60.96" width="0.1524" layer="91"/>
-<pinref part="P+10" gate="1" pin="+5V"/>
+<pinref part="SV1" gate="G$1" pin="1"/>
 </segment>
 </net>
@@
 <wire x1="87.63" y1="69.85" x2="113.03" y2="69.85" width="0.1524" layer="91"/>
 <label x="90.17" y="69.85" size="1.778" layer="95"/>
+<pinref part="SV1" gate="G$1" pin="3"/>
 </segment>
 </net>
@@
 <wire x1="90.17" y1="67.31" x2="113.03" y2="67.31" width="0.1524" layer="91"/>
 <label x="92.71" y="67.31" size="1.778" layer="95"/>
+<pinref part="SV1" gate="G$1" pin="4"/>
 </segment>
 </net>
@@
 <wire x1="107.95" y1="46.99" x2="118.11" y2="46.99" width="0.1524" layer="91"/>
 <label x="110.49" y="46.99" size="1.778" layer="95"/>
-</segment>
-<segment>
-<pinref part="X3" gate="-2" pin="K"/>
-<wire x1="191.77" y1="-1.27" x2="182.88" y2="-1.27" width="0.1524" layer="91"/>
-<label x="182.88" y="-1.27" size="1.778" layer="95"/>
+<pinref part="TP1" gate="G$1" pin="TP"/>
 </segment>
 </net>
@@
 <wire x1="107.95" y1="49.53" x2="118.11" y2="49.53" width="0.1524" layer="91"/>
 <label x="109.22" y="49.53" size="1.778" layer="95"/>
+<pinref part="TP2" gate="G$1" pin="TP"/>
 </segment>
 </net>
@@
 <wire x1="96.52" y1="-22.86" x2="100.33" y2="-22.86" width="0.1524" layer="91"/>
 <wire x1="100.33" y1="-22.86" x2="100.33" y2="-26.67" width="0.1524" layer="91"/>
-<wire x1="100.33" y1="-26.67" x2="127" y2="-26.67" width="0.1524" layer="91"/>
+<wire x1="100.33" y1="-26.67" x2="118.11" y2="-26.67" width="0.1524" layer="91"/>
 <pinref part="C6" gate="G$1" pin="2"/>
+<wire x1="118.11" y1="-26.67" x2="127" y2="-26.67" width="0.1524" layer="91"/>
 <wire x1="127" y1="-26.67" x2="191.77" y2="-26.67" width="0.1524" layer="91"/>
 <wire x1="127" y1="-24.13" x2="127" y2="-26.67" width="0.1524" layer="91"/>
@@
 <junction x="191.77" y="-26.67"/>
 <junction x="100.33" y="-22.86"/>
+<pinref part="TP5" gate="G$1" pin="TP"/>
+<junction x="118.11" y="-26.67"/>
 </segment>
 <segment>
@@
 <pinref part="R8" gate="G$1" pin="1"/>
 <pinref part="R9" gate="G$1" pin="2"/>
-<wire x1="146.05" y1="-35.56" x2="152.4" y2="-35.56" width="0.1524" layer="91"/>
+<wire x1="146.05" y1="-35.56" x2="149.86" y2="-35.56" width="0.1524" layer="91"/>
 <label x="147.32" y="-35.56" size="1.778" layer="95"/>
+<pinref part="TP4" gate="G$1" pin="TP"/>
+<wire x1="149.86" y1="-35.56" x2="152.4" y2="-35.56" width="0.1524" layer="91"/>
+<junction x="149.86" y="-35.56"/>
 </segment>
 <segment>
@@
 </segment>
 <segment>
-<pinref part="S1" gate="G$1" pin="NO"/>
-<wire x1="161.29" y1="72.39" x2="168.91" y2="72.39" width="0.1524" layer="91"/>
-<pinref part="R10" gate="G$1" pin="2"/>
-<label x="162.56" y="72.39" size="1.778" layer="95"/>
+<pinref part="SV1" gate="G$1" pin="5"/>
+<wire x1="113.03" y1="64.77" x2="100.33" y2="64.77" width="0.1524" layer="91"/>
+<label x="100.33" y="64.77" size="1.778" layer="95"/>
 </segment>
 </net>
@@
 </segment>
 <segment>
-<pinref part="S2" gate="G$1" pin="NO"/>
-<wire x1="161.29" y1="58.42" x2="168.91" y2="58.42" width="0.1524" layer="91"/>
-<pinref part="R11" gate="G$1" pin="2"/>
-<label x="162.56" y="58.42" size="1.778" layer="95"/>
+<pinref part="SV1" gate="G$1" pin="6"/>
+<wire x1="113.03" y1="62.23" x2="100.33" y2="62.23" width="0.1524" layer="91"/>
+<label x="100.33" y="62.23" size="1.778" layer="95"/>
 </segment>
 </net>
@@
 </segment>
 </net>
+<net name="N$11" class="0">
+<segment>
+<pinref part="X3" gate="-2" pin="K"/>
+<pinref part="TP3" gate="G$1" pin="TP"/>
+</segment>
+</net>

Commit message: Done with PCB Rev1 for Power Supply and Display PCB
Parts:
- added C13, C15, C17: 10u, rcl:C-USC0805
- added C14, C16, C18: 0.1u, rcl:C-USC0805
- added TP7: PTR1PAD1-20, testpad:PTR1PAD1-20
Connections:
- net +5V: now also C15.1, C16.1, C17.1, C18.1
- net 5: now also C13.1, C14.1, TP7.TP
- net GND: now also C13.2, C14.2, C15.2, C16.2, C17.2, C18.2
Other:
- moved on the sheet: C11, C12, D3, F1, LED2, R12, TP6, X1
