File: PCBdesign/teamNACHOrev1.brd (EAGLE design)
At the start: 100 x 80 mm, 47 parts, among them IC1 7805TV, Q2 TK40E06N1, Q3 TK40E06N1, U2 ATTINY85V-10SU, X2 1751248, X3 1751251

Commit message: hur ya go
asdfasdf
Parts:
- added C11: 10u, rcl:C0805
- added C12: 0.1u, rcl:C0805
- added LED2: (no value), eagle-ltspice:LED_LD260
- added R12: 470, rcl:M0805
- R8: value 100 -> 30k
- R9: value 100 -> 10k
- moved R11 249.3 mm to (66.7, 72.4), flipped to the bottom, turned to 180 degrees
- moved S2 229.3 mm to (63.5, 72.4)
- moved R9 188.9 mm to (64.8, 44.5), flipped to the bottom
- moved R10 186.5 mm to (67.3, 6.99), flipped to the bottom, turned to 180 degrees
- moved R8 179.8 mm to (64.8, 40.0), flipped to the bottom, turned to 180 degrees
- moved S1 159.9 mm to (63.5, 6.35)
- moved SV1 145.5 mm to (43.8, 42.5), turned to 90 degrees
- moved C10 141.2 mm to (12.7, 29.8), flipped to the bottom, turned to 90 degrees
- moved C9 134.1 mm to (20.3, 25.4), flipped to the bottom, turned to 90 degrees
- moved R6 133.5 mm to (39.4, 52.1), flipped to the bottom
- moved R7 128.6 mm to (45.7, 34.9), flipped to the bottom, turned to 90 degrees
- moved JP2 126.8 mm to (39.4, 30.5), turned to 270 degrees
- moved LED1 126.8 mm to (39.4, 48.9)
- moved IC1 112.5 mm to (15.2, 17.1), turned to 180 degrees
- moved U2 110.8 mm to (50.8, 29.2)
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Connections:
- removed net N$11: X2.2
- new net SCK-AT: JP2.3, U2.2
- net +5V: now also C11.1, C12.1
- net 5: now also R12.1
- net FB: now also R3.2, U$3.1, X2.1
- net GND: now also C11.2, C12.2, LED2.K; no longer OK1.2
- net GND_S: now also OK1.2, X2.2
- net N$8: now also U$3.3
- net N$9: now also LED2.A, R12.2; no longer R3.2, X2.1
- net VFB: now also U2.3; no longer JP2.3, U2.2
Routing:
- added copper zone on layer 1, net GND
- added copper zone on layer 16, net GND
Other:
- board size 100 x 80 mm -> 76.5 x 78.7 mm

Commit message: HERE YOU GO ADAM
Parts:
- removed R10, R11: 1k, rcl:R0805
- removed S1, S2: 5501, switch:5501
- added TP1, TP2, TP3, TP4, TP5, TP6: PTR1PAD1-20, testpad:P1-20
- SV1: device con-lstb:MA04-1 -> con-lsta:FE06
- moved SV1 88.1 mm to (8.26, -38.1), turned to 0 degrees
Connections:
- new net N$11: TP3.TP, X3.2
- net +5V: no longer S1.1A, S2.1A
- net FB-CGRD: now also TP2.TP
- net GND: now also TP6.TP; no longer R10.1, R11.1
- net GND_S: now also TP5.TP
- net LED-CLK: now also SV1.3
- net LED-DAT: now also SV1.4
- net PB_1: now also SV1.5; no longer R10.2, S1.NO
- net PB_2: now also SV1.6; no longer R11.2, S2.NO
- net POT: now also TP1.TP; no longer X3.2
- net VFB: now also TP4.TP
Changed lines of the file:
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@@
 <attribute name="NAME" x="34.925" y="34.29" size="1.27" layer="25" ratio="10" rot="R270"/>
-</element>
-<element name="SV1" library="con-lstb" package="MA04-1" value="" x="43.815" y="42.545" rot="R90">
-<attribute name="OC_NEWARK" value="unknown" x="43.815" y="42.545" size="1.778" layer="27" rot="R90" display="off"/>
-<attribute name="MF" value="" x="43.815" y="42.545" size="1.778" layer="27" rot="R90" display="off"/>
-<attribute name="MPN" value="" x="43.815" y="42.545" size="1.778" layer="27" rot="R90" display="off"/>
-<attribute name="OC_FARNELL" value="unknown" x="43.815" y="42.545" size="1.778" layer="27" rot="R90" display="off"/>
 </element>
 <element name="IC1" library="linear" package="TO220V" value="7805TV" x="15.24" y="17.145" smashed="yes" rot="R180">
@@
 <element name="R9" library="resistor" package="R0805" value="10k" x="64.77" y="44.45" smashed="yes" rot="MR0">
 <attribute name="NAME" x="65.405" y="45.72" size="1.27" layer="26" rot="MR0"/>
-</element>
-<element name="S1" library="switch" package="5501" value="5501" x="63.5" y="6.35" smashed="yes"/>
-<element name="S2" library="switch" package="5501" value="5501" x="63.5" y="72.39" smashed="yes"/>
-<element name="R10" library="rcl" package="R0805" value="1k" x="67.31" y="6.985" smashed="yes" rot="MR180">
-<attribute name="NAME" x="66.675" y="5.715" size="1.27" layer="26" rot="MR180"/>
-</element>
-<element name="R11" library="rcl" package="R0805" value="1k" x="66.675" y="72.39" smashed="yes" rot="MR180">
-<attribute name="NAME" x="66.04" y="71.12" size="1.27" layer="26" rot="MR180"/>
 </element>
 <element name="C11" library="rcl" package="C0805" value="10u" x="15.24" y="13.335" smashed="yes" rot="MR270">
@@
 </element>
 <element name="R12" library="rcl" package="M0805" value="470" x="3.175" y="21.59" rot="MR180"/>
+<element name="TP1" library="testpad" package="P1-20" value="PTR1PAD1-20" x="1.905" y="-4.445">
+<attribute name="TP_SIGNAL_NAME" value="" x="1.905" y="-4.445" size="1.778" layer="27" display="off"/>
+</element>
+<element name="TP2" library="testpad" package="P1-20" value="PTR1PAD1-20" x="1.905" y="-10.16">
+<attribute name="TP_SIGNAL_NAME" value="" x="1.905" y="-10.16" size="1.778" layer="27" display="off"/>
+</element>
+<element name="TP3" library="testpad" package="P1-20" value="PTR1PAD1-20" x="1.905" y="-15.875">
+<attribute name="TP_SIGNAL_NAME" value="" x="1.905" y="-15.875" size="1.778" layer="27" display="off"/>
+</element>
+<element name="TP4" library="testpad" package="P1-20" value="PTR1PAD1-20" x="1.905" y="-21.59">
+<attribute name="TP_SIGNAL_NAME" value="" x="1.905" y="-21.59" size="1.778" layer="27" display="off"/>
+</element>
+<element name="TP5" library="testpad" package="P1-20" value="PTR1PAD1-20" x="1.905" y="-27.305">
+<attribute name="TP_SIGNAL_NAME" value="" x="1.905" y="-27.305" size="1.778" layer="27" display="off"/>
+</element>
+<element name="TP6" library="testpad" package="P1-20" value="PTR1PAD1-20" x="1.905" y="-33.02">
+<attribute name="TP_SIGNAL_NAME" value="" x="1.905" y="-33.02" size="1.778" layer="27" display="off"/>
+</element>
+<element name="SV1" library="con-lsta" package="FE06" value="" x="8.255" y="-38.1">
+<attribute name="MPN" value="" x="8.255" y="-38.1" size="1.778" layer="27" display="off"/>
+<attribute name="OC_NEWARK" value="unknown" x="8.255" y="-38.1" size="1.778" layer="27" display="off"/>
+<attribute name="MF" value="" x="8.255" y="-38.1" size="1.778" layer="27" display="off"/>
+<attribute name="OC_FARNELL" value="unknown" x="8.255" y="-38.1" size="1.778" layer="27" display="off"/>
+</element>
 </elements>
 <signals>
@@
 <contactref element="Q3" pad="S"/>
 <contactref element="OK1" pad="4"/>
-<contactref element="SV1" pad="2"/>
-<contactref element="R10" pad="1"/>
-<contactref element="R11" pad="1"/>
 <polygon width="0.4064" layer="16">
 <vertex x="0" y="78.74"/>
@@
 <contactref element="C12" pad="2"/>
 <contactref element="LED2" pad="K"/>
+<contactref element="TP6" pad="TP"/>
+<contactref element="SV1" pad="2"/>
+<wire x1="1.905" y1="-33.02" x2="4.445" y2="-38.1" width="0" layer="19" extent="1-1"/>
+<wire x1="26.67" y1="2.54" x2="1.905" y2="-33.02" width="0" layer="19" extent="1-1"/>
 </signal>
 <signal name="N$2">
@@
 <contactref element="U$4" pad="1"/>
 <contactref element="R6" pad="1"/>
-<contactref element="SV1" pad="1"/>
-<contactref element="S1" pad="1A"/>
-<contactref element="S2" pad="1A"/>
 <contactref element="C11" pad="1"/>
 <contactref element="C12" pad="1"/>
-<wire x1="60.325" y1="61.28" x2="63.5" y2="76.2" width="0" layer="19" extent="16-16"/>
-<wire x1="59.69" y1="58.1" x2="60.325" y2="61.28" width="0" layer="19" extent="16-16"/>
+<contactref element="SV1" pad="1"/>
+<wire x1="59.69" y1="58.1" x2="72.49" y2="53.015" width="0" layer="19" extent="16-16"/>
+<wire x1="60.325" y1="61.28" x2="59.69" y2="58.1" width="0" layer="19" extent="16-16"/>
 <wire x1="56.515" y1="61.28" x2="60.325" y2="61.28" width="0" layer="19" extent="16-16"/>
 <wire x1="52.47" y1="60.1726" x2="56.515" y2="61.28" width="0" layer="19" extent="1-16"/>
@@
 <wire x1="40.32" y1="52.07" x2="50.07" y2="51.5874" width="0" layer="19" extent="1-16"/>
 <wire x1="40.64" y1="59.69" x2="40.32" y2="52.07" width="0" layer="19" extent="16-16"/>
-<wire x1="72.49" y1="53.015" x2="59.69" y2="58.1" width="0" layer="19" extent="16-16"/>
-<wire x1="43.815" y1="38.735" x2="40.32" y2="52.07" width="0" layer="19" extent="16-16"/>
-<wire x1="33.02" y1="17.78" x2="43.815" y2="38.735" width="0" layer="19" extent="1-1"/>
+<wire x1="33.02" y1="17.78" x2="40.32" y2="52.07" width="0" layer="19" extent="16-16"/>
 <wire x1="26.67" y1="17.78" x2="33.02" y2="17.78" width="0" layer="19" extent="1-1"/>
 <wire x1="20.32" y1="14.285" x2="26.67" y2="17.78" width="0" layer="19" extent="16-16"/>
 <wire x1="15.24" y1="14.285" x2="20.32" y2="14.285" width="0" layer="19" extent="16-16"/>
 <wire x1="9.4488" y1="14.3764" x2="15.24" y2="14.285" width="0" layer="19" extent="16-16"/>
-<wire x1="63.5" y1="10.16" x2="33.02" y2="17.78" width="0" layer="19" extent="1-1"/>
+<wire x1="1.905" y1="-38.1" x2="9.4488" y2="14.3764" width="0" layer="19" extent="1-1"/>
 </signal>
 <signal name="SCK">
@@
 <signal name="LED-CLK">
 <contactref element="U$1" pad="28"/>
+<contactref element="SV1" pad="3"/>
+<wire x1="6.985" y1="-38.1" x2="56.3626" y2="55.48" width="0" layer="19" extent="1-1"/>
 </signal>
 <signal name="LED-DAT">
 <contactref element="U$1" pad="27"/>
+<contactref element="SV1" pad="4"/>
+<wire x1="9.525" y1="-38.1" x2="56.3626" y2="54.68" width="0" layer="19" extent="1-1"/>
 </signal>
 <signal name="POT">
 <contactref element="U$1" pad="23"/>
-<contactref element="X3" pad="2"/>
-<wire x1="54.07" y1="51.5874" x2="72.49" y2="56.515" width="0" layer="19" extent="1-1"/>
+<contactref element="TP1" pad="TP"/>
+<wire x1="1.905" y1="-4.445" x2="54.07" y2="51.5874" width="0" layer="19" extent="1-1"/>
 </signal>
 <signal name="FB-CGRD">
 <contactref element="U$1" pad="24"/>
+<contactref element="TP2" pad="TP"/>
+<wire x1="1.905" y1="-10.16" x2="54.87" y2="51.5874" width="0" layer="19" extent="1-1"/>
 </signal>
 <signal name="N$5">
@@
 <contactref element="OK1" pad="2"/>
 <contactref element="X2" pad="2"/>
+<contactref element="TP5" pad="TP"/>
 <wire x1="65.72" y1="44.45" x2="72.49" y2="44.295" width="0" layer="19" extent="16-16"/>
 <wire x1="51.435" y1="38.735" x2="65.72" y2="44.45" width="0" layer="19" extent="16-16"/>
@@
 <wire x1="7.62" y1="69.85" x2="7.5946" y2="42.6466" width="0" layer="19" extent="1-1"/>
 <wire x1="42.225" y1="66.04" x2="51.435" y2="38.735" width="0" layer="19" extent="16-16"/>
+<wire x1="1.905" y1="-27.305" x2="15.24" y2="19.685" width="0" layer="19" extent="1-1"/>
 </signal>
 <signal name="VFB">
@@
 <contactref element="R9" pad="2"/>
 <contactref element="U2" pad="3"/>
+<contactref element="TP4" pad="TP"/>
 <wire x1="63.82" y1="40.005" x2="63.82" y2="44.45" width="0" layer="19" extent="16-16"/>
 <wire x1="47.0916" y1="28.575" x2="63.82" y2="40.005" width="0" layer="19" extent="1-16"/>
+<wire x1="1.905" y1="-21.59" x2="47.0916" y2="28.575" width="0" layer="19" extent="1-1"/>
 </signal>
 <signal name="PB_1">
 <contactref element="U$1" pad="11"/>
-<contactref element="S1" pad="NO"/>
-<contactref element="R10" pad="2"/>
-<wire x1="68.58" y1="10.16" x2="47.7774" y2="57.08" width="0" layer="19" extent="1-1"/>
-<wire x1="68.26" y1="6.985" x2="68.58" y2="10.16" width="0" layer="19" extent="16-16"/>
+<contactref element="SV1" pad="5"/>
+<wire x1="12.065" y1="-38.1" x2="47.7774" y2="57.08" width="0" layer="19" extent="1-1"/>
 </signal>
 <signal name="PB_2">
 <contactref element="U$1" pad="12"/>
-<contactref element="S2" pad="NO"/>
-<contactref element="R11" pad="2"/>
-<wire x1="67.625" y1="72.39" x2="68.58" y2="76.2" width="0" layer="19" extent="16-16"/>
-<wire x1="47.7774" y1="56.28" x2="67.625" y2="72.39" width="0" layer="19" extent="1-16"/>
+<contactref element="SV1" pad="6"/>
+<wire x1="14.605" y1="-38.1" x2="47.7774" y2="56.28" width="0" layer="19" extent="1-1"/>
 </signal>
 <signal name="OPTO">
@@
 <wire x1="4.125" y1="21.59" x2="5.715" y2="19.685" width="0" layer="19" extent="16-16"/>
 </signal>
+<signal name="N$11">
+<contactref element="X3" pad="2"/>
+<contactref element="TP3" pad="TP"/>
+<wire x1="1.905" y1="-15.875" x2="72.49" y2="56.515" width="0" layer="19" extent="1-1"/>
+</signal>
 </signals>

Commit message: dun
Parts:
- moved TP6 124.7 mm to (57.8, 78.4)
- moved TP5 121.4 mm to (61.6, 78.4)
- moved TP3 118.1 mm to (73.0, 78.4)
- moved SV1 117.8 mm to (39.4, 75.6), turned to 180 degrees
- moved TP2 109.0 mm to (65.4, 78.4)
- moved TP1 106.8 mm to (69.2, 78.4)
- moved TP4 96.7 mm to (66.7, 50.2)
- moved C10 45.8 mm to (57.8, 38.1)
- moved D3 45.6 mm to (65.4, 34.3), turned to 0 degrees
- moved IC1 40.8 mm to (47.6, 41.9), turned to 0 degrees
- moved U$4 37.0 mm to (56.4, 12.5)
- moved U$3 33.9 mm to (47.6, 43.2), turned to 180 degrees
- moved JP2 33.7 mm to (71.1, 41.9), turned to 90 degrees
- moved X1 30.7 mm to (67.3, 22.9)
- moved R3 30.5 mm to (56.5, 45.1), turned to 90 degrees
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Routing:
- net +5V: track 0.00 -> 116.0 mm, vias 0 -> 3
- net 5: track 0.00 -> 78.6 mm
- net PWM-C: track 0.00 -> 49.3 mm, vias 0 -> 1
- net N$5: track 0.00 -> 47.8 mm
- net PB_2: track 0.00 -> 42.4 mm
- net GND: track 0.00 -> 41.5 mm, vias 0 -> 1
- net PB_1: track 0.00 -> 37.9 mm
- net PWM-F: track 0.00 -> 36.0 mm, vias 0 -> 1
- net RESET: track 0.00 -> 35.2 mm, vias 0 -> 1
- net FB: track 0.00 -> 34.0 mm, vias 0 -> 2
- net N$20: track 0.00 -> 33.2 mm
- net N$7: track 0.00 -> 32.9 mm, vias 0 -> 1
- net N$17: track 0.00 -> 32.9 mm
- net N$14: track 0.00 -> 32.1 mm
- net LED-DAT: track 0.00 -> 31.5 mm
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- added copper zone on layer 16, net GND_S
- removed copper zone on layer 16, net GND
Other:
- board size 76.5 x 78.7 mm -> 76.5 x 66.3 mm

Commit message: Done with PCB Rev1 for Power Supply and Display PCB
Parts:
- added C13, C15, C17: 10u, rcl:C0805
- added C14, C16, C18: 0.1u, rcl:C0805
- added TP7: PTR1PAD1-20, testpad:P1-20
- moved C11 9.29 mm to (31.4, 18.4)
- moved C12 9.26 mm to (31.4, 21.9)
- moved X1 8.55 mm to (59.4, 26.0)
- moved LED2 7.62 mm to (14.0, 18.4)
- moved F1 7.49 mm to (71.4, 26.0), turned to 90 degrees
- moved U$4 7.38 mm to (49.7, 15.6)
- moved R2 3.31 mm to (13.0, 50.2)
- moved C5 3.24 mm to (17.1, 50.2)
- moved TP1 2.86 mm to (66.4, 78.4)
- moved TP2 2.86 mm to (62.5, 78.4)
- moved TP3 2.86 mm to (70.2, 78.4)
- moved TP5 2.86 mm to (58.7, 78.4)
- moved TP6 2.86 mm to (54.9, 78.4)
- moved D5 1.90 mm to (33.3, 32.4)
- moved D4 1.59 mm to (33.3, 35.6)
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Connections:
- net +5V: now also C15.1, C16.1, C17.1, C18.1
- net 5: now also C13.1, C14.1, TP7.TP
- net GND: now also C13.2, C14.2, C15.2, C16.2, C17.2, C18.2
Routing:
- net +5V: track 116.0 -> 167.3 mm
- net 5: track 78.6 -> 110.1 mm, vias 0 -> 2
- net GND: track 41.5 -> 69.0 mm
- net N$5: track 47.8 -> 22.1 mm
- net N$16: track 0.00 -> 16.6 mm
- net N$12: track 0.00 -> 11.9 mm
- net N$29: track 5.04 -> 16.8 mm
- net N$21: track 0.00 -> 10.2 mm
- net N$28: track 0.00 -> 7.62 mm
- net N$9: track 5.85 -> 12.2 mm
- net N$25: track 0.00 -> 5.33 mm
- net N$1: track 24.9 -> 29.1 mm
- net N$14: track 32.1 -> 36.2 mm
- net N$19: track 0.00 -> 3.14 mm
- net N$11: track 15.5 -> 13.0 mm
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Other:
- board text added: "--T$"
- board text added: "1:1 TXF"
- board text added: "1:1.5 TXF"
- board text added: "GND"
- board text added: "LED PCB"
- board text added: "NACHOpower, FALL 2015 ASH & NPC"
- board text added: "OUT"
- board text added: "TEST POINTS"
